File: uo_C_SE_Display_Module.brd (EAGLE design)
At the start: 35.5 x 26 mm, 14 parts, among them U1 UG-2864HSWEG01

Commit message: assembly process updates
Parts:
- added U$1, U$2, U$3: (no value), uo_C_SE_Library:FIDUCIAL
Other:
- board text added: "2019-03-13"
- board text added: "TD-OCSE-B-DM 2019-03-13"
- board text removed: "2018-05-08"
- board text removed: "TD-OCSE-B-DM 2018-05-08"
Changed lines of the file:
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@@
 <?xml version="1.0" encoding="utf-8"?>
 <!DOCTYPE eagle SYSTEM "eagle.dtd">
-<eagle version="9.0.1">
+<eagle version="9.3.1">
 <drawing>
 <settings>
@@
 <setting verticaltext="up"/>
 </settings>
-<grid distance="0.25" unitdist="mm" unit="mm" style="lines" multiple="1" display="yes" altdistance="0.05" altunitdist="mm" altunit="mm"/>
+<grid distance="0.5" unitdist="mm" unit="mm" style="lines" multiple="1" display="yes" altdistance="0.05" altunitdist="mm" altunit="mm"/>
 <layers>
 <layer number="1" name="Top" color="4" fill="1" visible="yes" active="yes"/>
-<layer number="2" name="Route2" color="1" fill="3" visible="no" active="no"/>
-<layer number="15" name="Route15" color="4" fill="6" visible="no" active="no"/>
 <layer number="16" name="Bottom" color="1" fill="1" visible="yes" active="yes"/>
 <layer number="17" name="Pads" color="2" fill="1" visible="yes" active="yes"/>
@@
 <wire x1="34.5" y1="26" x2="35.5" y2="25" width="0" layer="20" curve="-90"/>
 <text x="35" y="25.5" size="1.3" layer="22" ratio="10" rot="MR90" align="top-right">TD-OCSE-B-DM
-2018-05-08</text>
+2019-03-13</text>
 <text x="0.5" y="25.5" size="1.3" layer="22" ratio="10" rot="MR90" align="bottom-right">tall-dog.com
 CC BY-NC-SA 4.0</text>
@@
 <text x="2.65" y="4.25" size="1.3" layer="22" ratio="10" rot="MR270" align="bottom-center">GND</text>
 <text x="5.25" y="1.75" size="0.8" layer="21" ratio="10" rot="R180" align="center">TD-OCSE-B-DM</text>
-<text x="5.25" y="0.75" size="0.8" layer="21" ratio="10" rot="R180" align="center">2018-05-08</text>
+<text x="5.25" y="0.75" size="0.8" layer="21" ratio="10" rot="R180" align="center">2019-03-13</text>
 <text x="30.25" y="1.75" size="0.8" layer="21" ratio="10" rot="R180" align="center">CC BY-NC-SA 4.0</text>
 <text x="30.25" y="0.75" size="0.8" layer="21" ratio="10" rot="R180" align="center">tall-dog.com</text>
@@
 <param name="checkStop" value="1"/>
 <param name="checkValues" value="0"/>
+<param name="checkNames" value="1"/>
+<param name="checkWireStubs" value="1"/>
+<param name="checkPolygonWidth" value="0"/>
 <param name="useDiameter" value="13"/>
 <param name="maxErrors" value="50"/>
@@
 </autorouter>
 <elements>
-<element name="U1" library="uo_C_SE_Library" package="OLED-128X64" value="UG-2864HSWEG01" x="17.75" y="10"/>
+<element name="U1" library="uo_C_SE_Library" package="OLED-128X64" value="UG-2864HSWEG01" x="17.75" y="10" smashed="yes"/>
 <element name="R4" library="uo_C_SE_Library" package="0805-NP" value="10K" x="16.5" y="15" smashed="yes" rot="MR90">
 <attribute name="NAME" x="16.5" y="13" size="1" layer="22" ratio="10" rot="MR90" align="center-right"/>
@@
 <attribute name="NAME" x="31.25" y="8.4" size="1" layer="22" ratio="10" rot="SMR0" align="bottom-center"/>
 </element>
+<element name="U$1" library="uo_C_SE_Library" package="FIDUCIAL" value="" x="5.5" y="24" smashed="yes" rot="MR0"/>
+<element name="U$2" library="uo_C_SE_Library" package="FIDUCIAL" value="" x="30" y="24" smashed="yes" rot="MR0"/>
+<element name="U$3" library="uo_C_SE_Library" package="FIDUCIAL" value="" x="8.5" y="2" smashed="yes" rot="MR0"/>
 </elements>
 <signals>
@@
 <via x="33.25" y="17.25" extent="1-16" drill="0.35"/>
 <via x="1.75" y="15.75" extent="1-16" drill="0.35"/>
-<via x="5.75" y="24.5" extent="1-16" drill="0.35"/>
-<via x="29.25" y="24.5" extent="1-16" drill="0.35"/>
+<via x="7.25" y="25" extent="1-16" drill="0.35"/>
+<via x="28.25" y="25" extent="1-16" drill="0.35"/>
 <via x="1.75" y="19.5" extent="1-16" drill="0.35"/>
 <via x="33.25" y="21" extent="1-16" drill="0.35"/>
@@
 </signal>
 </signals>
+<mfgpreviewcolors>
+<mfgpreviewcolor name="soldermaskcolor" color="0xC8008000"/>
+<mfgpreviewcolor name="silkscreencolor" color="0xFFFEFEFE"/>
+<mfgpreviewcolor name="backgroundcolor" color="0xFF282828"/>
+<mfgpreviewcolor name="coppercolor" color="0xFFFFBF00"/>
+<mfgpreviewcolor name="substratecolor" color="0xFF786E46"/>
+</mfgpreviewcolors>
 </board>
 </drawing>
