File: uo_C_SE_Front_Panel.brd (EAGLE design)
At the start: 40.3 x 128.5 mm, 1 part

Commit message: assembly process updates
Other:
- board text added: "μo_C SE Front Panel TD-OCSE-B-FP CC BY-NC-SA 4.0 2019-03-24 tall-dog.com"
- board text removed: "μo_C SE Front Panel TD-OCSE-B-FP CC BY-NC-SA 4.0 2018-04-28 tall-dog.com"
Changed lines of the file:
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@@
 <?xml version="1.0" encoding="utf-8"?>
 <!DOCTYPE eagle SYSTEM "eagle.dtd">
-<eagle version="9.0.0">
+<eagle version="9.3.1">
 <drawing>
 <settings>
@@
 <layers>
 <layer number="1" name="Top" color="4" fill="1" visible="yes" active="yes"/>
-<layer number="2" name="Route2" color="1" fill="3" visible="no" active="no"/>
-<layer number="15" name="Route15" color="4" fill="6" visible="no" active="no"/>
 <layer number="16" name="Bottom" color="1" fill="1" visible="yes" active="yes"/>
 <layer number="17" name="Pads" color="2" fill="1" visible="yes" active="yes"/>
@@
 TD-OCSE-B-FP
 CC BY-NC-SA 4.0
-2018-04-28
+2019-03-24
 tall-dog.com</text>
 <text x="20.15" y="3" size="1.5" layer="29" ratio="10" align="center">CC BY-NC-SA 4.0</text>
@@
 <param name="checkStop" value="0"/>
 <param name="checkValues" value="0"/>
+<param name="checkNames" value="1"/>
+<param name="checkWireStubs" value="1"/>
+<param name="checkPolygonWidth" value="0"/>
 <param name="useDiameter" value="13"/>
 <param name="maxErrors" value="50"/>
@@
 </autorouter>
 <elements>
-<element name="E$1" library="uo_C_SE_Library" package="NEG-OUT" value="" x="32.65" y="58.5"/>
+<element name="E$1" library="uo_C_SE_Library" package="NEG-OUT" value="" x="32.65" y="58.5" smashed="yes"/>
 </elements>
 <signals>
@@
 </signal>
 </signals>
+<mfgpreviewcolors>
+<mfgpreviewcolor name="soldermaskcolor" color="0xC8008000"/>
+<mfgpreviewcolor name="silkscreencolor" color="0xFFFEFEFE"/>
+<mfgpreviewcolor name="backgroundcolor" color="0xFF282828"/>
+<mfgpreviewcolor name="coppercolor" color="0xFFFFBF00"/>
+<mfgpreviewcolor name="substratecolor" color="0xFF786E46"/>
+</mfgpreviewcolors>
 <errors>
 </errors>

Commit message: Revision C
Other:
- board text added: "TD-OCSE-C"
- board text added: "μo_C SE Front Panel TD-OCSE-C-FP/B CC BY-NC-SA 4.0 2020-02-22 tall-dog.com"
- board text removed: "Panel derived from work by Max Stadler (mxmxmx)"
- board text removed: "TD-OCSE-B"
- board text removed: "μo_C SE Front Panel TD-OCSE-B-FP CC BY-NC-SA 4.0 2019-03-24 tall-dog.com"
Changed lines of the file:
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@@
 <?xml version="1.0" encoding="utf-8"?>
 <!DOCTYPE eagle SYSTEM "eagle.dtd">
-<eagle version="9.3.1">
+<eagle version="9.5.2">
 <drawing>
 <settings>
@@
 <setting verticaltext="up"/>
 </settings>
-<grid distance="0.1" unitdist="mm" unit="mm" style="lines" multiple="1" display="yes" altdistance="0.025" altunitdist="inch" altunit="inch"/>
+<grid distance="0.5" unitdist="mm" unit="mm" style="lines" multiple="1" display="yes" altdistance="0.025" altunitdist="inch" altunit="inch"/>
 <layers>
 <layer number="1" name="Top" color="4" fill="1" visible="yes" active="yes"/>
@@
 <wire x1="31.8" y1="127.1" x2="33.8" y2="127.1" width="0" layer="20"/>
 <wire x1="31.8" y1="123.9" x2="33.8" y2="123.9" width="0" layer="20"/>
-<text x="20.15" y="127" size="1.5" layer="30" ratio="10" rot="MR0" align="top-center">μo_C SE
+<text x="20.15" y="126.5" size="1.6" layer="30" ratio="12" rot="MR0" align="top-center">μo_C SE
 Front Panel
-TD-OCSE-B-FP
+TD-OCSE-C-FP/B
 CC BY-NC-SA 4.0
-2019-03-24
+2020-02-22
 tall-dog.com</text>
 <text x="20.15" y="3" size="1.5" layer="29" ratio="10" align="center">CC BY-NC-SA 4.0</text>
-<text x="20.15" y="125.5" size="1.5" layer="29" ratio="10" align="center">TD-OCSE-B</text>
+<text x="20.15" y="125.5" size="1.5" layer="29" ratio="10" align="center">TD-OCSE-C</text>
 <wire x1="13.4" y1="127" x2="26.9" y2="127" width="0.15" layer="29"/>
 <wire x1="26.9" y1="127" x2="26.9" y2="124" width="0.15" layer="29"/>
@@
 <text x="20.15" y="58.5" size="2" layer="29" ratio="12" align="center">CV</text>
 <wire x1="7.65" y1="51" x2="7.65" y2="13.5" width="0.25" layer="29"/>
-<text x="20.15" y="88.5" size="1.5" layer="30" ratio="10" rot="MR0" align="center">Panel derived from work by
-Max Stadler (mxmxmx)</text>
 <rectangle x1="28.15" y1="10" x2="37.15" y2="57" layer="29"/>
 <wire x1="20.15" y1="51" x2="20.15" y2="13.5" width="0.25" layer="29"/>
