File: uo_C_SE_Main_Board.brd (EAGLE design)
At the start: 40 x 110.5 mm, 116 parts, among them J1 JACK-THONKICONN, J10 JACK-THONKICONN, J11 JACK-THONKICONN, J12 JACK-THONKICONN, J2 JACK-THONKICONN, J3 JACK-THONKICONN, J4 JACK-THONKICONN, J5 JACK-THONKICONN, J6 JACK-THONKICONN, J7 JACK-THONKICONN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

Commit message: assembly process updates
Routing:
- net SW-B: track 55.0 -> 69.4 mm
- net SW-T: track 35.8 -> 49.5 mm
- net CS-OLED: track 28.3 -> 19.7 mm, vias 0 -> 1
- net CS-DAC: track 35.9 -> 35.2 mm
- net RST-DAC: track 30.6 -> 31.3 mm
- net DOUT: track 41.6 -> 40.9 mm
- net CV-A: track 60.6 -> 61.1 mm
- net A3V3: track 104.3 -> 103.8 mm
Other:
- board text added: "2019-04-06"
- board text added: "TD-OCSE-B2-MB"
- board text removed: "2018-05-08"
- board text removed: "TD-OCSE-B-MB"

Commit message: Revision C
Parts:
- removed A2: (no value), uo_C_SE_Library:TEENSY-3.2-OUTLINE
- added U$4, U$5, U$6: (no value), uo_C_SE_Library:FIDUCIAL
- J1, J10, J11, J12, J2, J3, J4, J5, J6, J7, J8, J9: device uo_C_SE_Library:THONKICONN -> uo_C_SE_Library:JACK
- U$1: device uo_C_SE_Library:MARKING-CC-BY-NC-SA-4.0 -> uo_C_SE_Library:LOGO-CC
- U$2: device uo_C_SE_Library:MARKING-OSH-LOGO-5MM -> uo_C_SE_Library:LOGO-OSH
- U$3: device uo_C_SE_Library:MARKING-CC-LOGO -> uo_C_SE_Library:LOGO-REV
- moved U$3 32.8 mm to (10.0, 108.5)
- moved U$1 26.3 mm to (12.0, 75.5), turned to 0 degrees
- moved U$2 14.0 mm to (27.0, 69.0)
Other:
- board text added: "2020-02-22"
- board text added: "A2"
- board text added: "MAIN BOARD"
- board text added: "SN"
- board text added: "TD-OCSE-C-MB"
- board text added: "USB HERE"
- board text added: "tall-dog.com"
- board text removed: "2019-04-06"
- board text removed: "S/N"
- board text removed: "TALL-DOG.COM"
- board text removed: "TD-OCSE-B2-MB"
- board text removed: "USB PORT"
