File: uo_C_SE_Main_Board.sch (EAGLE design)
At the start: 112 parts, among them J1 JACK-THONKICONN, J10 JACK-THONKICONN, J11 JACK-THONKICONN, J12 JACK-THONKICONN, J2 JACK-THONKICONN, J3 JACK-THONKICONN, J4 JACK-THONKICONN, J5 JACK-THONKICONN, J6 JACK-THONKICONN, J7 JACK-THONKICONN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

Commit message: assembly process updates
Parts:
- A1: MANUFACTURERPARTNUMBER (none) -> TD-OCSE-B-DM
- C1, C12, C13, C14, C15, C16, C2, C20, C21, C31, C34, C5, C6, C7, C8: MANUFACTURERPARTNUMBER (none) -> CL10B104JB8NNNC
- C10, C11, C24, C25: MANUFACTURERPARTNUMBER (none) -> 865230440002
- C17, C18: MANUFACTURERPARTNUMBER (none) -> 865230443003
- C19, C23: MANUFACTURERPARTNUMBER (none) -> CL10B105KA8NNNC
- C22, C26, C32, C33: MANUFACTURERPARTNUMBER (none) -> CL10C220FB8NNWC
- C27, C28, C29, C30: MANUFACTURERPARTNUMBER (none) -> CL10C561JB8NNNC
- C3, C4, C9: MANUFACTURERPARTNUMBER (none) -> CL10B474KA8NFNC
- H1: MANUFACTURERPARTNUMBER (none) -> TSM-113-04-L-SV
- H2: MANUFACTURERPARTNUMBER (none) -> TSM-114-04-L-SV
- J1: MANUFACTURERPARTNUMBER (none) -> WQP-PJ398SM
- L1: MANUFACTURERPARTNUMBER (none) -> NLCV32T-100K-PFR
- R1: MANUFACTURERPARTNUMBER (none) -> ERJ-3EKF1002V
- R10, R11, R12, R13: MANUFACTURERPARTNUMBER (none) -> ERJ-3EKF7502V
- R14, R33, R34, R7: MANUFACTURERPARTNUMBER (none) -> ERJ-3EKF2200V
- R15, R16, R17, R18, R20, R21, R28, R36, R37, R38, R42, R8: MANUFACTURERPARTNUMBER (none) -> ERA-3AEB104V
- R19, R22, R23, R24, R25, R27, R35, R41: MANUFACTURERPARTNUMBER (none) -> ERJ-3EKF3302V
- R2, R3: MANUFACTURERPARTNUMBER (none) -> ERJ-3EKF4702V
- R26, R39, R40, R9: MANUFACTURERPARTNUMBER (none) -> ERA-3AEB2492V
- R29, R30, R31, R32: MANUFACTURERPARTNUMBER (none) -> ERJ-3EKF1000V
- R4, R5: MANUFACTURERPARTNUMBER (none) -> ERJ-3EKF5100V
- R6: MANUFACTURERPARTNUMBER (none) -> ERJ-3EKF2001V
- U1: MANUFACTURERPARTNUMBER (none) -> DAC8565IAPW

Commit message: Revision C
Other:
- note added: "C"
- note removed: "B"
Changed lines of the file:
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@@
 <?xml version="1.0" encoding="utf-8"?>
 <!DOCTYPE eagle SYSTEM "eagle.dtd">
-<eagle version="9.3.2">
+<eagle version="9.5.2">
 <drawing>
 <settings>
@@
 <grid distance="0.1" unitdist="inch" unit="inch" style="lines" multiple="1" display="no" altdistance="0.01" altunitdist="inch" altunit="inch"/>
 <layers>
+<layer number="1" name="Top" color="4" fill="1" visible="no" active="no"/>
+<layer number="2" name="Route2" color="1" fill="3" visible="no" active="no"/>
+<layer number="15" name="Route15" color="4" fill="6" visible="no" active="no"/>
+<layer number="16" name="Bottom" color="1" fill="1" visible="no" active="no"/>
+<layer number="17" name="Pads" color="2" fill="1" visible="no" active="no"/>
+<layer number="18" name="Vias" color="2" fill="1" visible="no" active="no"/>
+<layer number="19" name="Unrouted" color="6" fill="1" visible="no" active="no"/>
+<layer number="20" name="Dimension" color="24" fill="1" visible="no" active="no"/>
+<layer number="21" name="tPlace" color="7" fill="1" visible="no" active="no"/>
+<layer number="22" name="bPlace" color="14" fill="1" visible="no" active="no"/>
+<layer number="23" name="tOrigins" color="15" fill="1" visible="no" active="no"/>
+<layer number="24" name="bOrigins" color="15" fill="1" visible="no" active="no"/>
+<layer number="25" name="tNames" color="7" fill="1" visible="no" active="no"/>
+<layer number="26" name="bNames" color="7" fill="1" visible="no" active="no"/>
+<layer number="27" name="tValues" color="7" fill="1" visible="no" active="no"/>
+<layer number="28" name="bValues" color="7" fill="1" visible="no" active="no"/>
+<layer number="29" name="tStop" color="7" fill="3" visible="no" active="no"/>
+<layer number="30" name="bStop" color="7" fill="6" visible="no" active="no"/>
+<layer number="31" name="tCream" color="7" fill="4" visible="no" active="no"/>
+<layer number="32" name="bCream" color="7" fill="5" visible="no" active="no"/>
+<layer number="33" name="tFinish" color="6" fill="3" visible="no" active="no"/>
+<layer number="34" name="bFinish" color="6" fill="6" visible="no" active="no"/>
+<layer number="35" name="tGlue" color="7" fill="4" visible="no" active="no"/>
+<layer number="36" name="bGlue" color="7" fill="5" visible="no" active="no"/>
+<layer number="37" name="tTest" color="7" fill="1" visible="no" active="no"/>
+<layer number="38" name="bTest" color="7" fill="1" visible="no" active="no"/>
+<layer number="39" name="tKeepout" color="4" fill="11" visible="no" active="no"/>
+<layer number="40" name="bKeepout" color="1" fill="11" visible="no" active="no"/>
+<layer number="41" name="tRestrict" color="4" fill="10" visible="no" active="no"/>
+<layer number="42" name="bRestrict" color="1" fill="10" visible="no" active="no"/>
+<layer number="43" name="vRestrict" color="2" fill="10" visible="no" active="no"/>
+<layer number="44" name="Drills" color="7" fill="1" visible="no" active="no"/>
+<layer number="45" name="Holes" color="7" fill="1" visible="no" active="no"/>
+<layer number="46" name="Milling" color="3" fill="1" visible="no" active="no"/>
+<layer number="47" name="Measures" color="7" fill="1" visible="no" active="no"/>
+<layer number="48" name="Document" color="7" fill="1" visible="no" active="no"/>
+<layer number="49" name="Reference" color="7" fill="1" visible="no" active="no"/>
+<layer number="51" name="tDocu" color="11" fill="1" visible="no" active="no"/>
+<layer number="52" name="bDocu" color="7" fill="1" visible="no" active="no"/>
 <layer number="88" name="SimResults" color="9" fill="1" visible="yes" active="yes"/>
 <layer number="89" name="SimProbes" color="9" fill="1" visible="yes" active="yes"/>
@@
 Board derived from work by Max Stadler (mxmxmx)</text>
 <text x="148.59" y="6.35" size="2.54" layer="94">Website: tall-dog.com</text>
-<text x="236.22" y="6.35" size="3.81" layer="94">B</text>
+<text x="236.22" y="6.35" size="3.81" layer="94">C</text>
 <text x="179.07" y="11.43" size="2.54" layer="94">N/A</text>
 <text x="247.65" y="19.05" size="3.81" layer="94" align="center-right">Main Processing</text>
@@
 Board derived from work by Max Stadler (mxmxmx)</text>
 <text x="148.59" y="6.35" size="2.54" layer="94">Website: tall-dog.com</text>
-<text x="236.22" y="6.35" size="3.81" layer="94">B</text>
+<text x="236.22" y="6.35" size="3.81" layer="94">C</text>
 <text x="179.07" y="11.43" size="2.54" layer="94">N/A</text>
 <text x="247.65" y="19.05" size="3.81" layer="94" align="center-right">Analog I/O</text>
@@
 Board derived from work by Max Stadler (mxmxmx)</text>
 <text x="148.59" y="6.35" size="2.54" layer="94">Website: tall-dog.com</text>
-<text x="236.22" y="6.35" size="3.81" layer="94">B</text>
+<text x="236.22" y="6.35" size="3.81" layer="94">C</text>
 <text x="179.07" y="11.43" size="2.54" layer="94">N/A</text>
 <text x="247.65" y="19.05" size="3.81" layer="94" align="center-right">Power &amp; UI</text>
